File: decade.kicad_pcb (KiCad board)
At the start: 2 copper layers, 30 x 58 mm, 20 parts, among them J1 Conn_02x04_Odd_Even, J2 Conn_02x02_Odd_Even, J3 USB_B_Micro, J4 Conn_02x04_Odd_Even, SW1 SW_ROTARY_10_POS

Commit message: Minor updates including gerbers.
Parts:
- moved J4 26.8 mm to (128.0, 106.2), turned to 180 degrees
- moved J3 24.6 mm to (102.7, 102.5), turned to 270 degrees
Routing:
- net /IN: track 58.6 -> 70.2 mm, vias 3 -> 4
- net /THRU: track 18.2 -> 27.3 mm
- net +5V: track 128.8 -> 126.8 mm
- net GND: track 107.3 -> 108.3 mm, vias 4 -> 5
- net /OUT: vias 3 -> 2
